File: Breadboard Power Supply/KiCad/Schematic/Breadboard Power Supply.kicad_sch (KiCad schematic)
At the start: 17 parts, among them J1 Barrel_Jack_Switch, J2 Screw_Terminal_01x02, J3 Conn_01x03_Pin, J4 Conn_01x02_Pin, J5 Screw_Terminal_01x02, J6 Conn_01x02_Pin, J7 Conn_01x03_Pin, U1 LM317_TO-220, U2 LM7805_TO220

Commit message: Add files via upload
Connections:
- net PWR_OUT_TOP renamed PWR_OUTPUT_TOP
Other:
- note added: "3.3V Circuit"
- note removed: "3V Circuit"
Changed lines of the file:
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@@
 		)
 	)
-	(text "3V Circuit"
+	(text "3.3V Circuit"
 		(exclude_from_sim no)
 		(at 54.61 70.866 0)
@@
 		)
 	)
-	(label "PWR_OUT_TOP"
+	(label "PWR_OUTPUT_TOP"
 		(at 184.15 107.95 180)
 		(effects
